Commit message: modif for imu

File: install/spot_v1_description/share/spot_v1_description/urdf/spot_v1.xacro (robot description, xacro)
@@ -6,7 +6,7 @@
 <link name="base_link">
   <inertial>
-    <origin xyz="0.4744837095448095 0.23249999999999665 0.17036122042657198" rpy="0 0 0"/>
+    <origin xyz="3.3750779948604757e-15 0.0014661695131983521 0.17036122042657198" rpy="0 0 0"/>
     <mass value="4.569295440014468"/>
-    <inertia ixx="0.010005" iyy="0.064329" izz="0.069095" ixy="0.0" iyz="0.0" ixz="-0.000337"/>
+    <inertia ixx="0.064329" iyy="0.010005" izz="0.069095" ixy="-0.0" iyz="-0.000337" ixz="-0.0"/>
   </inertial>
   <visual>
@@ -26,10 +26,10 @@
 <link name="lower_fl_1">
   <inertial>
-    <origin xyz="0.043812108672994565 -0.0100340995070487 0.012048486431752617" rpy="0 0 0"/>
+    <origin xyz="0.0100340995070487 0.043812568641383415 0.012048486431752742" rpy="0 0 0"/>
     <mass value="0.03597522586843197"/>
-    <inertia ixx="4e-06" iyy="5.4e-05" izz="5e-05" ixy="-0.0" iyz="-0.0" ixz="-1.2e-05"/>
-  </inertial>
-  <visual>
-    <origin xyz="-0.628003 -0.336998 -0.086482" rpy="0 0 0"/>
+    <inertia ixx="5.4e-05" iyy="4e-06" izz="5e-05" ixy="0.0" iyz="-1.2e-05" ixz="0.0"/>
+  </inertial>
+  <visual>
+    <origin xyz="0.104498 -0.154985 -0.086482" rpy="0 0 0"/>
     <geometry>
       <mesh filename="file://$(find spot_v1_description)/meshes/lower_fl_1.stl" scale="0.001 0.001 0.001"/>
@@ -38,5 +38,5 @@
   </visual>
   <collision>
-    <origin xyz="-0.628003 -0.336998 -0.086482" rpy="0 0 0"/>
+    <origin xyz="0.104498 -0.154985 -0.086482" rpy="0 0 0"/>
     <geometry>
       <mesh filename="file://$(find spot_v1_description)/meshes/lower_fl_1.stl" scale="0.001 0.001 0.001"/>
@@ -46,10 +46,10 @@
 <link name="upper_fl_1">
   <inertial>
-    <origin xyz="0.01014350117997087 -0.0008587246147913064 -0.03708622546972476" rpy="0 0 0"/>
+    <origin xyz="0.0008587246147913619 0.010143961148359887 -0.03708622546972473" rpy="0 0 0"/>
     <mass value="0.03437614015191293"/>
-    <inertia ixx="3.3e-05" iyy="3.7e-05" izz="5e-06" ixy="-0.0" iyz="2e-06" ixz="9e-06"/>
-  </inertial>
-  <visual>
-    <origin xyz="-0.603554 -0.333998 -0.17" rpy="0 0 0"/>
+    <inertia ixx="3.7e-05" iyy="3.3e-05" izz="5e-06" ixy="0.0" iyz="9e-06" ixz="-2e-06"/>
+  </inertial>
+  <visual>
+    <origin xyz="0.101498 -0.130536 -0.17" rpy="0 0 0"/>
     <geometry>
       <mesh filename="file://$(find spot_v1_description)/meshes/upper_fl_1.stl" scale="0.001 0.001 0.001"/>
@@ -58,5 +58,5 @@
   </visual>
   <collision>
-    <origin xyz="-0.603554 -0.333998 -0.17" rpy="0 0 0"/>
+    <origin xyz="0.101498 -0.130536 -0.17" rpy="0 0 0"/>
     <geometry>
       <mesh filename="file://$(find spot_v1_description)/meshes/upper_fl_1.stl" scale="0.001 0.001 0.001"/>
@@ -66,10 +66,10 @@
 <link name="upper_bl_1">
   <inertial>
-    <origin xyz="0.010143880264565197 -0.0008587246147911398 -0.03708622546972459" rpy="0 0 0"/>
+    <origin xyz="0.0008587246147910704 0.010144340232953963 -0.03708622546972459" rpy="0 0 0"/>
     <mass value="0.03437614015191293"/>
-    <inertia ixx="3.3e-05" iyy="3.7e-05" izz="5e-06" ixy="-0.0" iyz="2e-06" ixz="9e-06"/>
-  </inertial>
-  <visual>
-    <origin xyz="-0.2935 -0.333998 -0.17" rpy="0 0 0"/>
+    <inertia ixx="3.7e-05" iyy="3.3e-05" izz="5e-06" ixy="0.0" iyz="9e-06" ixz="-2e-06"/>
+  </inertial>
+  <visual>
+    <origin xyz="0.101498 0.179518 -0.17" rpy="0 0 0"/>
     <geometry>
       <mesh filename="file://$(find spot_v1_description)/meshes/upper_bl_1.stl" scale="0.001 0.001 0.001"/>
@@ -78,5 +78,5 @@
   </visual>
   <collision>
-    <origin xyz="-0.2935 -0.333998 -0.17" rpy="0 0 0"/>
+    <origin xyz="0.101498 0.179518 -0.17" rpy="0 0 0"/>
     <geometry>
       <mesh filename="file://$(find spot_v1_description)/meshes/upper_bl_1.stl" scale="0.001 0.001 0.001"/>
@@ -86,10 +86,10 @@
 <link name="lower_bl_1">
   <inertial>
-    <origin xyz="0.0438124877575885 -0.010034099507049699 0.012048486431753158" rpy="0 0 0"/>
+    <origin xyz="0.01003409950704956 0.04381194772597723 0.012048486431753214" rpy="0 0 0"/>
     <mass value="0.03597522586843197"/>
-    <inertia ixx="4e-06" iyy="5.4e-05" izz="5e-05" ixy="-0.0" iyz="-0.0" ixz="-1.2e-05"/>
-  </inertial>
-  <visual>
-    <origin xyz="-0.317949 -0.336998 -0.086482" rpy="0 0 0"/>
+    <inertia ixx="5.4e-05" iyy="4e-06" izz="5e-05" ixy="0.0" iyz="-1.2e-05" ixz="0.0"/>
+  </inertial>
+  <visual>
+    <origin xyz="0.104498 0.155068 -0.086482" rpy="0 0 0"/>
     <geometry>
       <mesh filename="file://$(find spot_v1_description)/meshes/lower_bl_1.stl" scale="0.001 0.001 0.001"/>
@@ -98,5 +98,5 @@
   </visual>
   <collision>
-    <origin xyz="-0.317949 -0.336998 -0.086482" rpy="0 0 0"/>
+    <origin xyz="0.104498 0.155068 -0.086482" rpy="0 0 0"/>
     <geometry>
       <mesh filename="file://$(find spot_v1_description)/meshes/lower_bl_1.stl" scale="0.001 0.001 0.001"/>
@@ -106,10 +106,10 @@
 <link name="upper_fr_1">
   <inertial>
-    <origin xyz="0.010143486704232929 0.0008587229129283225 -0.03708620077467481" rpy="0 0 0"/>
+    <origin xyz="-0.0008587229129282392 0.010143946672621779 -0.03708620077467481" rpy="0 0 0"/>
     <mass value="0.03437614965320798"/>
-    <inertia ixx="3.3e-05" iyy="3.7e-05" izz="5e-06" ixy="0.0" iyz="-2e-06" ixz="9e-06"/>
-  </inertial>
-  <visual>
-    <origin xyz="-0.603554 -0.131002 -0.17" rpy="0 0 0"/>
+    <inertia ixx="3.7e-05" iyy="3.3e-05" izz="5e-06" ixy="-0.0" iyz="9e-06" ixz="2e-06"/>
+  </inertial>
+  <visual>
+    <origin xyz="-0.101498 -0.130536 -0.17" rpy="0 0 0"/>
     <geometry>
       <mesh filename="file://$(find spot_v1_description)/meshes/upper_fr_1.stl" scale="0.001 0.001 0.001"/>
@@ -118,5 +118,5 @@
   </visual>
   <collision>
-    <origin xyz="-0.603554 -0.131002 -0.17" rpy="0 0 0"/>
+    <origin xyz="-0.101498 -0.130536 -0.17" rpy="0 0 0"/>
     <geometry>
       <mesh filename="file://$(find spot_v1_description)/meshes/upper_fr_1.stl" scale="0.001 0.001 0.001"/>
@@ -126,10 +126,10 @@
 <link name="upper_br_1">
   <inertial>
-    <origin xyz="0.01014386578882781 0.0008587229129282947 -0.037086200774674116" rpy="0 0 0"/>
+    <origin xyz="-0.0008587229129282947 0.010144325757216577 -0.037086200774674116" rpy="0 0 0"/>
     <mass value="0.03437614965320798"/>
-    <inertia ixx="3.3e-05" iyy="3.7e-05" izz="5e-06" ixy="0.0" iyz="-2e-06" ixz="9e-06"/>
-  </inertial>
-  <visual>
-    <origin xyz="-0.2935 -0.131002 -0.17" rpy="0 0 0"/>
+    <inertia ixx="3.7e-05" iyy="3.3e-05" izz="5e-06" ixy="-0.0" iyz="9e-06" ixz="2e-06"/>
+  </inertial>
+  <visual>
+    <origin xyz="-0.101498 0.179518 -0.17" rpy="0 0 0"/>
     <geometry>
       <mesh filename="file://$(find spot_v1_description)/meshes/upper_br_1.stl" scale="0.001 0.001 0.001"/>
@@ -138,5 +138,5 @@
   </visual>
   <collision>
-    <origin xyz="-0.2935 -0.131002 -0.17" rpy="0 0 0"/>
+    <origin xyz="-0.101498 0.179518 -0.17" rpy="0 0 0"/>
     <geometry>
       <mesh filename="file://$(find spot_v1_description)/meshes/upper_br_1.stl" scale="0.001 0.001 0.001"/>
@@ -146,10 +146,10 @@
 <link name="lower_fr_1">
   <inertial>
-    <origin xyz="0.04381216258027687 0.010034098184056067 0.012048585657918914" rpy="0 0 0"/>
+    <origin xyz="-0.010034098184055942 0.04381262254866572 0.012048585657918914" rpy="0 0 0"/>
     <mass value="0.03597520460150114"/>
-    <inertia ixx="4e-06" iyy="5.4e-05" izz="5e-05" ixy="0.0" iyz="0.0" ixz="-1.2e-05"/>
-  </inertial>
-  <visual>
-    <origin xyz="-0.628003 -0.128002 -0.086482" rpy="0 0 0"/>
+    <inertia ixx="5.4e-05" iyy="4e-06" izz="5e-05" ixy="-0.0" iyz="-1.2e-05" ixz="-0.0"/>
+  </inertial>
+  <visual>
+    <origin xyz="-0.104498 -0.154985 -0.086482" rpy="0 0 0"/>
     <geometry>
       <mesh filename="file://$(find spot_v1_description)/meshes/lower_fr_1.stl" scale="0.001 0.001 0.001"/>
@@ -158,5 +158,5 @@
   </visual>
   <collision>
-    <origin xyz="-0.628003 -0.128002 -0.086482" rpy="0 0 0"/>
+    <origin xyz="-0.104498 -0.154985 -0.086482" rpy="0 0 0"/>
     <geometry>
       <mesh filename="file://$(find spot_v1_description)/meshes/lower_fr_1.stl" scale="0.001 0.001 0.001"/>
@@ -166,10 +166,10 @@
 <link name="lower_br_1">
   <inertial>
-    <origin xyz="0.04381254166487092 0.010034098184056706 0.012048585657919789" rpy="0 0 0"/>
+    <origin xyz="-0.010034098184056664 0.04381200163325967 0.012048585657919789" rpy="0 0 0"/>
     <mass value="0.03597520460150114"/>
-    <inertia ixx="4e-06" iyy="5.4e-05" izz="5e-05" ixy="0.0" iyz="0.0" ixz="-1.2e-05"/>
-  </inertial>
-  <visual>
-    <origin xyz="-0.317949 -0.128002 -0.086482" rpy="0 0 0"/>
+    <inertia ixx="5.4e-05" iyy="4e-06" izz="5e-05" ixy="-0.0" iyz="-1.2e-05" ixz="-0.0"/>
+  </inertial>
+  <visual>
+    <origin xyz="-0.104498 0.155068 -0.086482" rpy="0 0 0"/>
     <geometry>
       <mesh filename="file://$(find spot_v1_description)/meshes/lower_br_1.stl" scale="0.001 0.001 0.001"/>
@@ -178,5 +178,5 @@
   </visual>
   <collision>
-    <origin xyz="-0.317949 -0.128002 -0.086482" rpy="0 0 0"/>
+    <origin xyz="-0.104498 0.155068 -0.086482" rpy="0 0 0"/>
     <geometry>
       <mesh filename="file://$(find spot_v1_description)/meshes/lower_br_1.stl" scale="0.001 0.001 0.001"/>
@@ -186,10 +186,10 @@
 <link name="elbow_bl_5">
   <inertial>
-    <origin xyz="0.008500000000042363 0.005346701893651606 -1.6653345369377348e-16" rpy="0 0 0"/>
+    <origin xyz="-0.005346701893651634 0.008500459968431101 -8.326672684688674e-17" rpy="0 0 0"/>
     <mass value="0.008194856226231374"/>
-    <inertia ixx="1e-06" iyy="0.0" izz="1e-06" ixy="-0.0" iyz="0.0" ixz="0.0"/>
-  </inertial>
-  <visual>
-    <origin xyz="-0.285 -0.295 -0.17" rpy="0 0 0"/>
+    <inertia ixx="0.0" iyy="1e-06" izz="1e-06" ixy="0.0" iyz="0.0" ixz="-0.0"/>
+  </inertial>
+  <visual>
+    <origin xyz="0.0625 0.188018 -0.17" rpy="0 0 0"/>
     <geometry>
       <mesh filename="file://$(find spot_v1_description)/meshes/elbow_bl_5.stl" scale="0.001 0.001 0.001"/>
@@ -198,5 +198,5 @@
   </visual>
   <collision>
-    <origin xyz="-0.285 -0.295 -0.17" rpy="0 0 0"/>
+    <origin xyz="0.0625 0.188018 -0.17" rpy="0 0 0"/>
     <geometry>
       <mesh filename="file://$(find spot_v1_description)/meshes/elbow_bl_5.stl" scale="0.001 0.001 0.001"/>
@@ -206,10 +206,10 @@
 <link name="elbow_fl_1">
   <inertial>
-    <origin xyz="-0.008500379084552478 0.005346701893651606 0.0" rpy="0 0 0"/>
+    <origin xyz="-0.005346701893651551 -0.008499919116163546 0.0" rpy="0 0 0"/>
     <mass value="0.008194856226231374"/>
-    <inertia ixx="1e-06" iyy="0.0" izz="1e-06" ixy="-0.0" iyz="0.0" ixz="-0.0"/>
-  </inertial>
-  <visual>
-    <origin xyz="-0.612054 -0.295 -0.17" rpy="0 0 0"/>
+    <inertia ixx="0.0" iyy="1e-06" izz="1e-06" ixy="0.0" iyz="0.0" ixz="0.0"/>
+  </inertial>
+  <visual>
+    <origin xyz="0.0625 -0.139036 -0.17" rpy="0 0 0"/>
     <geometry>
       <mesh filename="file://$(find spot_v1_description)/meshes/elbow_fl_1.stl" scale="0.001 0.001 0.001"/>
@@ -218,5 +218,5 @@
   </visual>
   <collision>
-    <origin xyz="-0.612054 -0.295 -0.17" rpy="0 0 0"/>
+    <origin xyz="0.0625 -0.139036 -0.17" rpy="0 0 0"/>
     <geometry>
       <mesh filename="file://$(find spot_v1_description)/meshes/elbow_fl_1.stl" scale="0.001 0.001 0.001"/>
@@ -226,10 +226,10 @@
 <link name="elbow_br_1">
   <inertial>
-    <origin xyz="0.008500000000042252 -0.005346701893651523 0.0" rpy="0 0 0"/>
+    <origin xyz="0.005346701893651509 0.00850045996843099 0.0" rpy="0 0 0"/>
     <mass value="0.008194856226231374"/>
-    <inertia ixx="1e-06" iyy="0.0" izz="1e-06" ixy="0.0" iyz="0.0" ixz="0.0"/>
-  </inertial>
-  <visual>
-    <origin xyz="-0.285 -0.17 -0.17" rpy="0 0 0"/>
+    <inertia ixx="0.0" iyy="1e-06" izz="1e-06" ixy="-0.0" iyz="0.0" ixz="0.0"/>
+  </inertial>
+  <visual>
+    <origin xyz="-0.0625 0.188018 -0.17" rpy="0 0 0"/>
     <geometry>
       <mesh filename="file://$(find spot_v1_description)/meshes/elbow_br_1.stl" scale="0.001 0.001 0.001"/>
@@ -238,5 +238,5 @@
   </visual>
   <collision>
-    <origin xyz="-0.285 -0.17 -0.17" rpy="0 0 0"/>
+    <origin xyz="-0.0625 0.188018 -0.17" rpy="0 0 0"/>
     <geometry>
       <mesh filename="file://$(find spot_v1_description)/meshes/elbow_br_1.stl" scale="0.001 0.001 0.001"/>
@@ -246,10 +246,10 @@
 <link name="elbow_fr_1">
   <inertial>
-    <origin xyz="-0.008500379084552478 -0.005346701893651523 0.0" rpy="0 0 0"/>
+    <origin xyz="0.005346701893651579 -0.008499919116163601 0.0" rpy="0 0 0"/>
     <mass value="0.008194856226231374"/>
-    <inertia ixx="1e-06" iyy="0.0" izz="1e-06" ixy="0.0" iyz="0.0" ixz="0.0"/>
-  </inertial>
-  <visual>
-    <origin xyz="-0.612054 -0.17 -0.17" rpy="0 0 0"/>
+    <inertia ixx="0.0" iyy="1e-06" izz="1e-06" ixy="-0.0" iyz="0.0" ixz="0.0"/>
+  </inertial>
+  <visual>
+    <origin xyz="-0.0625 -0.139036 -0.17" rpy="0 0 0"/>
     <geometry>
       <mesh filename="file://$(find spot_v1_description)/meshes/elbow_fr_1.stl" scale="0.001 0.001 0.001"/>
@@ -258,5 +258,5 @@
   </visual>
   <collision>
-    <origin xyz="-0.612054 -0.17 -0.17" rpy="0 0 0"/>
+    <origin xyz="-0.0625 -0.139036 -0.17" rpy="0 0 0"/>
     <geometry>
       <mesh filename="file://$(find spot_v1_description)/meshes/elbow_fr_1.stl" scale="0.001 0.001 0.001"/>
@@ -264,87 +264,137 @@
   </collision>
 </link>
+<link name="base_laser_1">
+  <inertial>
+    <origin xyz="7.105427357601002e-17 2.7042609146085694e-07 0.00987517472943178" rpy="0 0 0"/>
+    <mass value="0.03571195095111218"/>
+    <inertia ixx="5e-06" iyy="5e-06" izz="6e-06" ixy="0.0" iyz="0.0" ixz="0.0"/>
+  </inertial>
+  <visual>
+    <origin xyz="-0.0 0.024491 -0.215" rpy="0 0 0"/>
+    <geometry>
+      <mesh filename="file://$(find spot_v1_description)/meshes/base_laser_1.stl" scale="0.001 0.001 0.001"/>
+    </geometry>
+    <material name="silver"/>
+  </visual>
+  <collision>
+    <origin xyz="-0.0 0.024491 -0.215" rpy="0 0 0"/>
+    <geometry>
+      <mesh filename="file://$(find spot_v1_description)/meshes/base_laser_1.stl" scale="0.001 0.001 0.001"/>
+    </geometry>
+  </collision>
+</link>
+<link name="base_imu">
+  <inertial>
+    <origin xyz="3.552713678800501e-17 2.7042609152677644e-07 -0.0024999999999999883" rpy="0 0 0"/>
+    <mass value="0.0008185"/>
+    <inertia ixx="0.0" iyy="0.0" izz="0.0" ixy="-0.0" iyz="-0.0" ixz="0.0"/>
+  </inertial>
+  <visual>
+    <origin xyz="-0.0 0.024491 -0.125" rpy="0 0 0"/>
+    <geometry>
+      <mesh filename="file://$(find spot_v1_description)/meshes/base_imu.stl" scale="0.001 0.001 0.001"/>
+    </geometry>
+    <material name="silver"/>
+  </visual>
+  <collision>
+    <origin xyz="-0.0 0.024491 -0.125" rpy="0 0 0"/>
+    <geometry>
+      <mesh filename="file://$(find spot_v1_description)/meshes/base_imu.stl" scale="0.001 0.001 0.001"/>
+    </geometry>
+  </collision>
+</link>
 <joint name="Revolute 29" type="revolute">
-  <origin xyz="0.024449 0.003 -0.083518" rpy="0 0 0"/>
+  <origin xyz="-0.003 0.024449 -0.083518" rpy="0 0 0"/>
   <parent link="upper_fl_1"/>
   <child link="lower_fl_1"/>
-  <axis xyz="0.0 -1.0 -0.0"/>
+  <axis xyz="1.0 -0.0 -0.0"/>
   <limit upper="0.785398" lower="-0.872665" effort="100" velocity="100"/>
 </joint>
 <joint name="Revolute 30" type="revolute">
-  <origin xyz="-0.0085 0.038998 0.0" rpy="0 0 0"/>
+  <origin xyz="-0.038998 -0.0085 0.0" rpy="0 0 0"/>
   <parent link="elbow_fl_1"/>
   <child link="upper_fl_1"/>
-  <axis xyz="0.0 1.0 0.0"/>
+  <axis xyz="-1.0 0.0 0.0"/>
   <limit upper="3.316126" lower="0.523599" effort="100" velocity="100"/>
 </joint>
 <joint name="Revolute 32" type="revolute">
-  <origin xyz="0.0085 0.038998 0.0" rpy="0 0 0"/>
+  <origin xyz="-0.038998 0.0085 0.0" rpy="0 0 0"/>
   <parent link="elbow_bl_5"/>
   <child link="upper_bl_1"/>
-  <axis xyz="-0.0 1.0 0.0"/>
+  <axis xyz="-1.0 0.0 0.0"/>
   <limit upper="3.316126" lower="0.523599" effort="100" velocity="100"/>
 </joint>
 <joint name="Revolute 33" type="revolute">
-  <origin xyz="0.024449 0.003 -0.083518" rpy="0 0 0"/>
+  <origin xyz="-0.003 0.02445 -0.083518" rpy="0 0 0"/>
   <parent link="upper_bl_1"/>
   <child link="lower_bl_1"/>
-  <axis xyz="-0.0 1.0 0.0"/>
+  <axis xyz="-1.0 0.0 0.0"/>
   <limit upper="0.785398" lower="-0.872665" effort="100" velocity="100"/>
 </joint>
 <joint name="Revolute 35" type="revolute">
-  <origin xyz="-0.0085 -0.038998 0.0" rpy="0 0 0"/>
+  <origin xyz="0.038998 -0.0085 0.0" rpy="0 0 0"/>
   <parent link="elbow_fr_1"/>
   <child link="upper_fr_1"/>
-  <axis xyz="0.0 -1.0 0.0"/>
+  <axis xyz="1.0 -0.0 0.0"/>
   <limit upper="-0.523599" lower="-3.316126" effort="100" velocity="100"/>
 </joint>
 <joint name="Revolute 36" type="revolute">
-  <origin xyz="0.0085 -0.038998 0.0" rpy="0 0 0"/>
+  <origin xyz="0.038998 0.0085 0.0" rpy="0 0 0"/>
   <parent link="elbow_br_1"/>
   <child link="upper_br_1"/>
-  <axis xyz="0.0 -1.0 0.0"/>
+  <axis xyz="1.0 -0.0 0.0"/>
   <limit upper="-0.523599" lower="-3.316126" effort="100" velocity="100"/>
 </joint>
 <joint name="Revolute 37" type="revolute">
-  <origin xyz="0.024449 -0.003 -0.083518" rpy="0 0 0"/>
+  <origin xyz="0.003 0.024449 -0.083518" rpy="0 0 0"/>
   <parent link="upper_fr_1"/>
   <child link="lower_fr_1"/>
-  <axis xyz="0.0 -1.0 -0.0"/>
+  <axis xyz="1.0 -0.0 -0.0"/>
   <limit upper="0.785398" lower="-0.872665" effort="100" velocity="100"/>
 </joint>
 <joint name="Revolute 38" type="revolute">
-  <origin xyz="0.024449 -0.003 -0.083518" rpy="0 0 0"/>
+  <origin xyz="0.003 0.02445 -0.083518" rpy="0 0 0"/>
   <parent link="upper_br_1"/>
   <child link="lower_br_1"/>
-  <axis xyz="-0.0 1.0 -0.0"/>
+  <axis xyz="-1.0 0.0 -0.0"/>
   <limit upper="0.785398" lower="-0.872665" effort="100" velocity="100"/>
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
File: src/spot_v1_description/urdf/spot_v1.xacro (robot description, xacro)
@@ -284,5 +284,5 @@
   </collision>
 </link>
-<link name="base_imu_1">
+<link name="base_imu">
   <inertial>
     <origin xyz="3.552713678800501e-17 2.7042609152677644e-07 -0.0024999999999999883" rpy="0 0 0"/>
@@ -293,5 +293,5 @@
     <origin xyz="-0.0 0.024491 -0.125" rpy="0 0 0"/>
     <geometry>
-      <mesh filename="file://$(find spot_v1_description)/meshes/base_imu_1.stl" scale="0.001 0.001 0.001"/>
+      <mesh filename="file://$(find spot_v1_description)/meshes/base_imu.stl" scale="0.001 0.001 0.001"/>
     </geometry>
     <material name="silver"/>
@@ -300,5 +300,5 @@
     <origin xyz="-0.0 0.024491 -0.125" rpy="0 0 0"/>
     <geometry>
-      <mesh filename="file://$(find spot_v1_description)/meshes/base_imu_1.stl" scale="0.001 0.001 0.001"/>
+      <mesh filename="file://$(find spot_v1_description)/meshes/base_imu.stl" scale="0.001 0.001 0.001"/>
     </geometry>
   </collision>
@@ -396,5 +396,5 @@
   <origin xyz="0.0 -0.024491 0.125" rpy="0 0 0"/>
   <parent link="base_link"/>
-  <child link="base_imu_1"/>
+  <child link="base_imu"/>
 </joint>
 </robot>
