Commit message: updated urdf

File: src/spot_v1_description/urdf/spot_v1.xacro (robot description, xacro)
@@ -6,7 +6,7 @@
 <link name="base_link">
   <inertial>
-    <origin xyz="0.473770936725285 0.23249999999999724 0.170342087630803" rpy="0 0 0"/>
-    <mass value="4.824853924420272"/>
-    <inertia ixx="0.010566" iyy="0.073453" izz="0.078475" ixy="0.0" iyz="0.0" ixz="-0.000338"/>
+    <origin xyz="0.4744837095448095 0.23249999999999665 0.17036122042657198" rpy="0 0 0"/>
+    <mass value="4.569295440014468"/>
+    <inertia ixx="0.010005" iyy="0.064329" izz="0.069095" ixy="0.0" iyz="0.0" ixz="-0.000337"/>
   </inertial>
   <visual>
@@ -26,10 +26,10 @@
 <link name="lower_fl_1">
   <inertial>
-    <origin xyz="0.041054614081095675 -0.010034099507048977 0.019473751887917543" rpy="0 0 0"/>
+    <origin xyz="0.043812108672994565 -0.0100340995070487 0.012048486431752617" rpy="0 0 0"/>
     <mass value="0.03597522586843197"/>
-    <inertia ixx="1e-05" iyy="5.4e-05" izz="4.5e-05" ixy="-0.0" iyz="-0.0" ixz="-1.9e-05"/>
-  </inertial>
-  <visual>
-    <origin xyz="-0.604134 -0.336998 -0.091996" rpy="0 0 0"/>
+    <inertia ixx="4e-06" iyy="5.4e-05" izz="5e-05" ixy="-0.0" iyz="-0.0" ixz="-1.2e-05"/>
+  </inertial>
+  <visual>
+    <origin xyz="-0.628003 -0.336998 -0.086482" rpy="0 0 0"/>
     <geometry>
       <mesh filename="file://$(find spot_v1_description)/meshes/lower_fl_1.stl" scale="0.001 0.001 0.001"/>
@@ -38,5 +38,5 @@
   </visual>
   <collision>
-    <origin xyz="-0.604134 -0.336998 -0.091996" rpy="0 0 0"/>
+    <origin xyz="-0.628003 -0.336998 -0.086482" rpy="0 0 0"/>
     <geometry>
       <mesh filename="file://$(find spot_v1_description)/meshes/lower_fl_1.stl" scale="0.001 0.001 0.001"/>
@@ -46,10 +46,10 @@
 <link name="upper_fl_1">
   <inertial>
-    <origin xyz="0.01642934831494003 -0.0008587246147913064 -0.03476133605013029" rpy="0 0 0"/>
+    <origin xyz="0.01014350117997087 -0.0008587246147913064 -0.03708622546972476" rpy="0 0 0"/>
     <mass value="0.03437614015191293"/>
-    <inertia ixx="2.9e-05" iyy="3.7e-05" izz="9e-06" ixy="-1e-06" iyz="2e-06" ixz="1.3e-05"/>
-  </inertial>
-  <visual>
-    <origin xyz="-0.565554 -0.333998 -0.17" rpy="0 0 0"/>
+    <inertia ixx="3.3e-05" iyy="3.7e-05" izz="5e-06" ixy="-0.0" iyz="2e-06" ixz="9e-06"/>
+  </inertial>
+  <visual>
+    <origin xyz="-0.603554 -0.333998 -0.17" rpy="0 0 0"/>
     <geometry>
       <mesh filename="file://$(find spot_v1_description)/meshes/upper_fl_1.stl" scale="0.001 0.001 0.001"/>
@@ -58,5 +58,5 @@
   </visual>
   <collision>
-    <origin xyz="-0.565554 -0.333998 -0.17" rpy="0 0 0"/>
+    <origin xyz="-0.603554 -0.333998 -0.17" rpy="0 0 0"/>
     <geometry>
       <mesh filename="file://$(find spot_v1_description)/meshes/upper_fl_1.stl" scale="0.001 0.001 0.001"/>
@@ -66,10 +66,10 @@
 <link name="upper_bl_1">
   <inertial>
-    <origin xyz="0.016429727399533856 -0.0008587246147911398 -0.03476133605013032" rpy="0 0 0"/>
+    <origin xyz="0.010143880264565197 -0.0008587246147911398 -0.03708622546972459" rpy="0 0 0"/>
     <mass value="0.03437614015191293"/>
-    <inertia ixx="2.9e-05" iyy="3.7e-05" izz="9e-06" ixy="-1e-06" iyz="2e-06" ixz="1.3e-05"/>
-  </inertial>
-  <visual>
-    <origin xyz="-0.3135 -0.333998 -0.17" rpy="0 0 0"/>
+    <inertia ixx="3.3e-05" iyy="3.7e-05" izz="5e-06" ixy="-0.0" iyz="2e-06" ixz="9e-06"/>
+  </inertial>
+  <visual>
+    <origin xyz="-0.2935 -0.333998 -0.17" rpy="0 0 0"/>
     <geometry>
       <mesh filename="file://$(find spot_v1_description)/meshes/upper_bl_1.stl" scale="0.001 0.001 0.001"/>
@@ -78,5 +78,5 @@
   </visual>
   <collision>
-    <origin xyz="-0.3135 -0.333998 -0.17" rpy="0 0 0"/>
+    <origin xyz="-0.2935 -0.333998 -0.17" rpy="0 0 0"/>
     <geometry>
       <mesh filename="file://$(find spot_v1_description)/meshes/upper_bl_1.stl" scale="0.001 0.001 0.001"/>
@@ -86,10 +86,10 @@
 <link name="lower_bl_1">
   <inertial>
-    <origin xyz="0.041054993165689446 -0.010034099507049699 0.01947375188791821" rpy="0 0 0"/>
+    <origin xyz="0.0438124877575885 -0.010034099507049699 0.012048486431753158" rpy="0 0 0"/>
     <mass value="0.03597522586843197"/>
-    <inertia ixx="1e-05" iyy="5.4e-05" izz="4.5e-05" ixy="-0.0" iyz="-0.0" ixz="-1.9e-05"/>
-  </inertial>
-  <visual>
-    <origin xyz="-0.35208 -0.336998 -0.091996" rpy="0 0 0"/>
+    <inertia ixx="4e-06" iyy="5.4e-05" izz="5e-05" ixy="-0.0" iyz="-0.0" ixz="-1.2e-05"/>
+  </inertial>
+  <visual>
+    <origin xyz="-0.317949 -0.336998 -0.086482" rpy="0 0 0"/>
     <geometry>
       <mesh filename="file://$(find spot_v1_description)/meshes/lower_bl_1.stl" scale="0.001 0.001 0.001"/>
@@ -98,5 +98,5 @@
   </visual>
   <collision>
-    <origin xyz="-0.35208 -0.336998 -0.091996" rpy="0 0 0"/>
+    <origin xyz="-0.317949 -0.336998 -0.086482" rpy="0 0 0"/>
     <geometry>
       <mesh filename="file://$(find spot_v1_description)/meshes/lower_bl_1.stl" scale="0.001 0.001 0.001"/>
@@ -106,10 +106,10 @@
 <link name="upper_fr_1">
   <inertial>
-    <origin xyz="0.016429329770870527 0.0008587229129283225 -0.034761314243939245" rpy="0 0 0"/>
+    <origin xyz="0.010143486704232929 0.0008587229129283225 -0.03708620077467481" rpy="0 0 0"/>
     <mass value="0.03437614965320798"/>
-    <inertia ixx="2.9e-05" iyy="3.7e-05" izz="9e-06" ixy="1e-06" iyz="-2e-06" ixz="1.3e-05"/>
-  </inertial>
-  <visual>
-    <origin xyz="-0.565554 -0.131002 -0.17" rpy="0 0 0"/>
+    <inertia ixx="3.3e-05" iyy="3.7e-05" izz="5e-06" ixy="0.0" iyz="-2e-06" ixz="9e-06"/>
+  </inertial>
+  <visual>
+    <origin xyz="-0.603554 -0.131002 -0.17" rpy="0 0 0"/>
     <geometry>
       <mesh filename="file://$(find spot_v1_description)/meshes/upper_fr_1.stl" scale="0.001 0.001 0.001"/>
@@ -118,5 +118,5 @@
   </visual>
   <collision>
-    <origin xyz="-0.565554 -0.131002 -0.17" rpy="0 0 0"/>
+    <origin xyz="-0.603554 -0.131002 -0.17" rpy="0 0 0"/>
     <geometry>
       <mesh filename="file://$(find spot_v1_description)/meshes/upper_fr_1.stl" scale="0.001 0.001 0.001"/>
@@ -126,10 +126,10 @@
 <link name="upper_br_1">
   <inertial>
-    <origin xyz="0.01642970885546491 0.000858722912928267 -0.03476131424393847" rpy="0 0 0"/>
+    <origin xyz="0.01014386578882781 0.0008587229129282947 -0.037086200774674116" rpy="0 0 0"/>
     <mass value="0.03437614965320798"/>
-    <inertia ixx="2.9e-05" iyy="3.7e-05" izz="9e-06" ixy="1e-06" iyz="-2e-06" ixz="1.3e-05"/>
-  </inertial>
-  <visual>
-    <origin xyz="-0.3135 -0.131002 -0.17" rpy="0 0 0"/>
+    <inertia ixx="3.3e-05" iyy="3.7e-05" izz="5e-06" ixy="0.0" iyz="-2e-06" ixz="9e-06"/>
+  </inertial>
+  <visual>
+    <origin xyz="-0.2935 -0.131002 -0.17" rpy="0 0 0"/>
     <geometry>
       <mesh filename="file://$(find spot_v1_description)/meshes/upper_br_1.stl" scale="0.001 0.001 0.001"/>
@@ -138,5 +138,5 @@
   </visual>
   <collision>
-    <origin xyz="-0.3135 -0.131002 -0.17" rpy="0 0 0"/>
+    <origin xyz="-0.2935 -0.131002 -0.17" rpy="0 0 0"/>
     <geometry>
       <mesh filename="file://$(find spot_v1_description)/meshes/upper_br_1.stl" scale="0.001 0.001 0.001"/>
@@ -146,10 +146,10 @@
 <link name="lower_fr_1">
   <inertial>
-    <origin xyz="0.04105464993896191 0.010034098184056234 0.019473858967516952" rpy="0 0 0"/>
+    <origin xyz="0.04381216258027687 0.010034098184056067 0.012048585657918914" rpy="0 0 0"/>
     <mass value="0.03597520460150114"/>
-    <inertia ixx="1e-05" iyy="5.4e-05" izz="4.5e-05" ixy="0.0" iyz="0.0" ixz="-1.9e-05"/>
-  </inertial>
-  <visual>
-    <origin xyz="-0.604134 -0.128002 -0.091996" rpy="0 0 0"/>
+    <inertia ixx="4e-06" iyy="5.4e-05" izz="5e-05" ixy="0.0" iyz="0.0" ixz="-1.2e-05"/>
+  </inertial>
+  <visual>
+    <origin xyz="-0.628003 -0.128002 -0.086482" rpy="0 0 0"/>
     <geometry>
       <mesh filename="file://$(find spot_v1_description)/meshes/lower_fr_1.stl" scale="0.001 0.001 0.001"/>
@@ -158,5 +158,5 @@
   </visual>
   <collision>
-    <origin xyz="-0.604134 -0.128002 -0.091996" rpy="0 0 0"/>
+    <origin xyz="-0.628003 -0.128002 -0.086482" rpy="0 0 0"/>
     <geometry>
       <mesh filename="file://$(find spot_v1_description)/meshes/lower_fr_1.stl" scale="0.001 0.001 0.001"/>
@@ -166,10 +166,10 @@
 <link name="lower_br_1">
   <inertial>
-    <origin xyz="0.04105502902355568 0.010034098184056706 0.019473858967517438" rpy="0 0 0"/>
+    <origin xyz="0.04381254166487092 0.010034098184056706 0.012048585657919789" rpy="0 0 0"/>
     <mass value="0.03597520460150114"/>
-    <inertia ixx="1e-05" iyy="5.4e-05" izz="4.5e-05" ixy="0.0" iyz="0.0" ixz="-1.9e-05"/>
-  </inertial>
-  <visual>
-    <origin xyz="-0.35208 -0.128002 -0.091996" rpy="0 0 0"/>
+    <inertia ixx="4e-06" iyy="5.4e-05" izz="5e-05" ixy="0.0" iyz="0.0" ixz="-1.2e-05"/>
+  </inertial>
+  <visual>
+    <origin xyz="-0.317949 -0.128002 -0.086482" rpy="0 0 0"/>
     <geometry>
       <mesh filename="file://$(find spot_v1_description)/meshes/lower_br_1.stl" scale="0.001 0.001 0.001"/>
@@ -178,5 +178,5 @@
   </visual>
   <collision>
-    <origin xyz="-0.35208 -0.128002 -0.091996" rpy="0 0 0"/>
+    <origin xyz="-0.317949 -0.128002 -0.086482" rpy="0 0 0"/>
     <geometry>
       <mesh filename="file://$(find spot_v1_description)/meshes/lower_br_1.stl" scale="0.001 0.001 0.001"/>
@@ -184,41 +184,41 @@
   </collision>
 </link>
-<link name="elbow_fl_1">
-  <inertial>
-    <origin xyz="0.008499620915447537 0.005346701893651606 0.0" rpy="0 0 0"/>
+<link name="elbow_bl_5">
+  <inertial>
+    <origin xyz="0.008500000000042363 0.005346701893651606 -1.6653345369377348e-16" rpy="0 0 0"/>
     <mass value="0.008194856226231374"/>
     <inertia ixx="1e-06" iyy="0.0" izz="1e-06" ixy="-0.0" iyz="0.0" ixz="0.0"/>
   </inertial>
   <visual>
-    <origin xyz="-0.557054 -0.295 -0.17" rpy="0 0 0"/>
-    <geometry>
-      <mesh filename="file://$(find spot_v1_description)/meshes/elbow_fl_1.stl" scale="0.001 0.001 0.001"/>
-    </geometry>
-    <material name="silver"/>
-  </visual>
-  <collision>
-    <origin xyz="-0.557054 -0.295 -0.17" rpy="0 0 0"/>
-    <geometry>
-      <mesh filename="file://$(find spot_v1_description)/meshes/elbow_fl_1.stl" scale="0.001 0.001 0.001"/>
-    </geometry>
-  </collision>
-</link>
-<link name="elbow_bl_5">
-  <inertial>
-    <origin xyz="0.008500000000042307 0.005346701893651606 -1.6653345369377348e-16" rpy="0 0 0"/>
+    <origin xyz="-0.285 -0.295 -0.17" rpy="0 0 0"/>
+    <geometry>
+      <mesh filename="file://$(find spot_v1_description)/meshes/elbow_bl_5.stl" scale="0.001 0.001 0.001"/>
+    </geometry>
+    <material name="silver"/>
+  </visual>
+  <collision>
+    <origin xyz="-0.285 -0.295 -0.17" rpy="0 0 0"/>
+    <geometry>
+      <mesh filename="file://$(find spot_v1_description)/meshes/elbow_bl_5.stl" scale="0.001 0.001 0.001"/>
+    </geometry>
+  </collision>
+</link>
+<link name="elbow_fl_1">
+  <inertial>
+    <origin xyz="-0.008500379084552478 0.005346701893651606 0.0" rpy="0 0 0"/>
     <mass value="0.008194856226231374"/>
     <inertia ixx="1e-06" iyy="0.0" izz="1e-06" ixy="-0.0" iyz="0.0" ixz="-0.0"/>
   </inertial>
   <visual>
-    <origin xyz="-0.305 -0.295 -0.17" rpy="0 0 0"/>
-    <geometry>
-      <mesh filename="file://$(find spot_v1_description)/meshes/elbow_bl_5.stl" scale="0.001 0.001 0.001"/>
-    </geometry>
-    <material name="silver"/>
-  </visual>
-  <collision>
-    <origin xyz="-0.305 -0.295 -0.17" rpy="0 0 0"/>
-    <geometry>
-      <mesh filename="file://$(find spot_v1_description)/meshes/elbow_bl_5.stl" scale="0.001 0.001 0.001"/>
+    <origin xyz="-0.612054 -0.295 -0.17" rpy="0 0 0"/>
+    <geometry>
+      <mesh filename="file://$(find spot_v1_description)/meshes/elbow_fl_1.stl" scale="0.001 0.001 0.001"/>
+    </geometry>
+    <material name="silver"/>
+  </visual>
+  <collision>
+    <origin xyz="-0.612054 -0.295 -0.17" rpy="0 0 0"/>
+    <geometry>
+      <mesh filename="file://$(find spot_v1_description)/meshes/elbow_fl_1.stl" scale="0.001 0.001 0.001"/>
     </geometry>
   </collision>
@@ -231,5 +231,5 @@
   </inertial>
   <visual>
-    <origin xyz="-0.305 -0.17 -0.17" rpy="0 0 0"/>
+    <origin xyz="-0.285 -0.17 -0.17" rpy="0 0 0"/>
     <geometry>
       <mesh filename="file://$(find spot_v1_description)/meshes/elbow_br_1.stl" scale="0.001 0.001 0.001"/>
@@ -238,5 +238,5 @@
   </visual>
   <collision>
-    <origin xyz="-0.305 -0.17 -0.17" rpy="0 0 0"/>
+    <origin xyz="-0.285 -0.17 -0.17" rpy="0 0 0"/>
     <geometry>
       <mesh filename="file://$(find spot_v1_description)/meshes/elbow_br_1.stl" scale="0.001 0.001 0.001"/>
@@ -246,10 +246,10 @@
 <link name="elbow_fr_1">
   <inertial>
-    <origin xyz="0.008499620915447537 -0.005346701893651523 0.0" rpy="0 0 0"/>
+    <origin xyz="-0.008500379084552478 -0.005346701893651523 0.0" rpy="0 0 0"/>
     <mass value="0.008194856226231374"/>
     <inertia ixx="1e-06" iyy="0.0" izz="1e-06" ixy="0.0" iyz="0.0" ixz="0.0"/>
   </inertial>
   <visual>
-    <origin xyz="-0.557054 -0.17 -0.17" rpy="0 0 0"/>
+    <origin xyz="-0.612054 -0.17 -0.17" rpy="0 0 0"/>
     <geometry>
       <mesh filename="file://$(find spot_v1_description)/meshes/elbow_fr_1.stl" scale="0.001 0.001 0.001"/>
@@ -258,5 +258,5 @@
   </visual>
   <collision>
-    <origin xyz="-0.557054 -0.17 -0.17" rpy="0 0 0"/>
+    <origin xyz="-0.612054 -0.17 -0.17" rpy="0 0 0"/>
     <geometry>
       <mesh filename="file://$(find spot_v1_description)/meshes/elbow_fr_1.stl" scale="0.001 0.001 0.001"/>
@@ -265,5 +265,5 @@
 </link>
 <joint name="Revolute 29" type="revolute">
-  <origin xyz="0.03858 0.003 -0.078004" rpy="0 0 0"/>
+  <origin xyz="0.024449 0.003 -0.083518" rpy="0 0 0"/>
   <parent link="upper_fl_1"/>
   <child link="lower_fl_1"/>
@@ -272,9 +272,9 @@
 </joint>
 <joint name="Revolute 30" type="revolute">
-  <origin xyz="0.0085 0.038998 0.0" rpy="0 0 0"/>
+  <origin xyz="-0.0085 0.038998 0.0" rpy="0 0 0"/>
   <parent link="elbow_fl_1"/>
   <child link="upper_fl_1"/>
   <axis xyz="0.0 1.0 0.0"/>
-  <limit upper="3.316126" lower="0.349066" effort="100" velocity="100"/>
+  <limit upper="3.316126" lower="0.523599" effort="100" velocity="100"/>
 </joint>
 <joint name="Revolute 32" type="revolute">
@@ -283,19 +283,19 @@
   <child link="upper_bl_1"/>
   <axis xyz="-0.0 1.0 0.0"/>
-  <limit upper="3.316126" lower="0.349066" effort="100" velocity="100"/>
+  <limit upper="3.316126" lower="0.523599" effort="100" velocity="100"/>
 </joint>
 <joint name="Revolute 33" type="revolute">
-  <origin xyz="0.03858 0.003 -0.078004" rpy="0 0 0"/>
+  <origin xyz="0.024449 0.003 -0.083518" rpy="0 0 0"/>
   <parent link="upper_bl_1"/>
   <child link="lower_bl_1"/>
-  <axis xyz="0.0 1.0 0.0"/>
+  <axis xyz="-0.0 1.0 0.0"/>
   <limit upper="0.785398" lower="-0.872665" effort="100" velocity="100"/>
 </joint>
 <joint name="Revolute 35" type="revolute">
-  <origin xyz="0.0085 -0.038998 0.0" rpy="0 0 0"/>
+  <origin xyz="-0.0085 -0.038998 0.0" rpy="0 0 0"/>
   <parent link="elbow_fr_1"/>
   <child link="upper_fr_1"/>
   <axis xyz="0.0 -1.0 0.0"/>
-  <limit upper="-0.349066" lower="-3.316126" effort="100" velocity="100"/>
+  <limit upper="-0.523599" lower="-3.316126" effort="100" velocity="100"/>
 </joint>
 <joint name="Revolute 36" type="revolute">
@@ -304,8 +304,8 @@
   <child link="upper_br_1"/>
   <axis xyz="0.0 -1.0 0.0"/>
-  <limit upper="-0.349066" lower="-3.316126" effort="100" velocity="100"/>
+  <limit upper="-0.523599" lower="-3.316126" effort="100" velocity="100"/>
 </joint>
 <joint name="Revolute 37" type="revolute">
-  <origin xyz="0.03858 -0.003 -0.078004" rpy="0 0 0"/>
+  <origin xyz="0.024449 -0.003 -0.083518" rpy="0 0 0"/>
   <parent link="upper_fr_1"/>
   <child link="lower_fr_1"/>
@@ -314,5 +314,5 @@
 </joint>
 <joint name="Revolute 38" type="revolute">
-  <origin xyz="0.03858 -0.003 -0.078004" rpy="0 0 0"/>
+  <origin xyz="0.024449 -0.003 -0.083518" rpy="0 0 0"/>
   <parent link="upper_br_1"/>
   <child link="lower_br_1"/>
@@ -320,29 +320,30 @@
   <limit upper="0.785398" lower="-0.872665" effort="100" velocity="100"/>
 </joint>
-<joint name="Revolute 39" type="revolute">
-  <origin xyz="0.557054 0.295 0.17" rpy="0 0 0"/>
+<joint name="Revolute 43" type="revolute">
+  <origin xyz="0.285 0.295 0.17" rpy="0 0 0"/>
+  <parent link="base_link"/>
+  <child link="elbow_bl_5"/>
+  <axis xyz="1.0 0.0 0.0"/>
+  <limit upper="1.570796" lower="-1.570796" effort="100" velocity="100"/>
+</joint>
+<joint name="Revolute 45" type="revolute">
+  <origin xyz="0.612054 0.295 0.17" rpy="0 0 0"/>
   <parent link="base_link"/>
   <child link="elbow_fl_1"/>
-  <axis xyz="-1.0 0.0 0.0"/>
+  <axis xyz="1.0 0.0 0.0"/>
   <limit upper="1.570796" lower="-1.570796" effort="100" velocity="100"/>
 </joint>
-<joint name="Revolute 40" type="revolute">
-  <origin xyz="0.305 0.295 0.17" rpy="0 0 0"/>
-  <parent link="base_link"/>
-  <child link="elbow_bl_5"/>
-  <axis xyz="-1.0 0.0 0.0"/>
-  <limit upper="1.570796" lower="-1.570796" effort="100" velocity="100"/>
-</joint>
-<joint name="Revolute 41" type="continuous">
-  <origin xyz="0.305 0.17 0.17" rpy="0 0 0"/>
+<joint name="Revolute 46" type="revolute">
+  <origin xyz="0.285 0.17 0.17" rpy="0 0 0"/>
   <parent link="base_link"/>
   <child link="elbow_br_1"/>
   <axis xyz="-1.0 0.0 0.0"/>
-</joint>
-<joint name="Revolute 42" type="revolute">
-  <origin xyz="0.557054 0.17 0.17" rpy="0 0 0"/>
+  <limit upper="1.570796" lower="-1.570796" effort="100" velocity="100"/>
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
Commit message: modif imu

File: src/spot_v1_description/urdf/spot_v1.xacro (robot description, xacro)
@@ -24,4 +24,32 @@
   </collision>
 </link>
+<!-- Adjusted LIDAR link and joint -->
+<link name="base_laser">
+  <inertial>
+    <origin xyz="0 0 0" rpy="0 0 0"/>
+    <mass value="0.1"/>
+    <inertia ixx="0.001" iyy="0.001" izz="0.001" ixy="0.0" iyz="0.0" ixz="0.0"/>
+  </inertial>
+  <visual>
+    <origin xyz="0 0 0" rpy="0 0 0"/>
+    <geometry>
+      <cylinder length="0.1" radius="0.05"/>
+    </geometry>
+    <material name="gray">
+      <color rgba="0.5 0.5 0.5 1.0"/>
+    </material>
+  </visual>
+  <collision>
+    <origin xyz="0 0 0" rpy="0 0 0"/>
+    <geometry>
+      <cylinder length="0.1" radius="0.05"/>
+    </geometry>
+  </collision>
+</link>
+<joint name="base_laser_joint" type="fixed">
+  <parent link="base_link"/>
+  <child link="base_laser"/>
+  <origin xyz="0.1 0 0.1" rpy="0 0 0"/>
+</joint>
 <link name="lower_fl_1">
   <inertial>

Commit message: inverted two axis in urdf

File: src/spot_v1_description/urdf/spot_v1.xacro (robot description, xacro)
@@ -329,5 +329,5 @@
   <parent link="upper_bl_1"/>
   <child link="lower_bl_1"/>
-  <axis xyz="-1.0 0.0 0.0"/>
+  <axis xyz="1.0 -0.0 -0.0"/>
   <limit upper="0.785398" lower="-0.872665" effort="100" velocity="100"/>
 </joint>
@@ -378,5 +378,5 @@
   <parent link="base_link"/>
   <child link="elbow_br_1"/>
-  <axis xyz="0.0 1.0 0.0"/>
+  <axis xyz="0.0 -1.0 0.0"/>
   <limit upper="1.570796" lower="-1.570796" effort="100" velocity="100"/>
 </joint>
