Commit message: fixed mass/inertia in spot description

File: src/spot_v1_description/urdf/spot_v1.xacro (robot description, xacro)
@@ -7,6 +7,6 @@
   <inertial>
     <origin xyz="3.3750779948604757e-15 0.0014661695131983521 0.17036122042657198" rpy="0 0 0"/>
-    <mass value="4.569295440014468"/>
-    <inertia ixx="0.064329" iyy="0.010005" izz="0.069095" ixy="-0.0" iyz="-0.000337" ixz="-0.0"/>
+    <mass value="1.5"/>
+    <inertia ixx="0.015" iyy="0.035" izz="0.045" ixy="0" ixz="0" iyz="0"/>
   </inertial>
   <visual>
@@ -27,6 +27,6 @@
   <inertial>
     <origin xyz="0.0100340995070487 0.043812568641383415 0.012048486431752742" rpy="0 0 0"/>
-    <mass value="0.03597522586843197"/>
-    <inertia ixx="5.4e-05" iyy="4e-06" izz="5e-05" ixy="0.0" iyz="-1.2e-05" ixz="0.0"/>
+    <mass value="0.02"/>
+    <inertia ixx="0.00005" iyy="0.00005" izz="0.00001" ixy="0" ixz="0" iyz="0"/>
   </inertial>
   <visual>
@@ -47,6 +47,6 @@
   <inertial>
     <origin xyz="0.0008587246147913619 0.010143961148359887 -0.03708622546972473" rpy="0 0 0"/>
-    <mass value="0.03437614015191293"/>
-    <inertia ixx="3.7e-05" iyy="3.3e-05" izz="5e-06" ixy="0.0" iyz="9e-06" ixz="-2e-06"/>
+    <mass value="0.06"/>
+    <inertia ixx="0.0001" iyy="0.0001" izz="0.00005" ixy="0" ixz="0" iyz="0"/>
   </inertial>
   <visual>
@@ -67,6 +67,6 @@
   <inertial>
     <origin xyz="0.0008587246147910704 0.010144340232953963 -0.03708622546972459" rpy="0 0 0"/>
-    <mass value="0.03437614015191293"/>
-    <inertia ixx="3.7e-05" iyy="3.3e-05" izz="5e-06" ixy="0.0" iyz="9e-06" ixz="-2e-06"/>
+    <mass value="0.06"/>
+    <inertia ixx="0.0001" iyy="0.0001" izz="0.00005" ixy="0" ixz="0" iyz="0"/>
   </inertial>
   <visual>
@@ -87,6 +87,6 @@
   <inertial>
     <origin xyz="0.01003409950704956 0.04381194772597723 0.012048486431753214" rpy="0 0 0"/>
-    <mass value="0.03597522586843197"/>
-    <inertia ixx="5.4e-05" iyy="4e-06" izz="5e-05" ixy="0.0" iyz="-1.2e-05" ixz="0.0"/>
+    <mass value="0.02"/>
+    <inertia ixx="0.00005" iyy="0.00005" izz="0.00001" ixy="0" ixz="0" iyz="0"/>
   </inertial>
   <visual>
@@ -107,6 +107,6 @@
   <inertial>
     <origin xyz="-0.0008587229129282392 0.010143946672621779 -0.03708620077467481" rpy="0 0 0"/>
-    <mass value="0.03437614965320798"/>
-    <inertia ixx="3.7e-05" iyy="3.3e-05" izz="5e-06" ixy="-0.0" iyz="9e-06" ixz="2e-06"/>
+    <mass value="0.06"/>
+    <inertia ixx="0.0001" iyy="0.0001" izz="0.00005" ixy="0" ixz="0" iyz="0"/>
   </inertial>
   <visual>
@@ -127,6 +127,6 @@
   <inertial>
     <origin xyz="-0.0008587229129282947 0.010144325757216577 -0.037086200774674116" rpy="0 0 0"/>
-    <mass value="0.03437614965320798"/>
-    <inertia ixx="3.7e-05" iyy="3.3e-05" izz="5e-06" ixy="-0.0" iyz="9e-06" ixz="2e-06"/>
+    <mass value="0.06"/>
+    <inertia ixx="0.0001" iyy="0.0001" izz="0.00005" ixy="0" ixz="0" iyz="0"/>
   </inertial>
   <visual>
@@ -147,6 +147,6 @@
   <inertial>
     <origin xyz="-0.010034098184055942 0.04381262254866572 0.012048585657918914" rpy="0 0 0"/>
-    <mass value="0.03597520460150114"/>
-    <inertia ixx="5.4e-05" iyy="4e-06" izz="5e-05" ixy="-0.0" iyz="-1.2e-05" ixz="-0.0"/>
+    <mass value="0.02"/>
+    <inertia ixx="0.00005" iyy="0.00005" izz="0.00001" ixy="0" ixz="0" iyz="0"/>
   </inertial>
   <visual>
@@ -167,6 +167,6 @@
   <inertial>
     <origin xyz="-0.010034098184056664 0.04381200163325967 0.012048585657919789" rpy="0 0 0"/>
-    <mass value="0.03597520460150114"/>
-    <inertia ixx="5.4e-05" iyy="4e-06" izz="5e-05" ixy="-0.0" iyz="-1.2e-05" ixz="-0.0"/>
+    <mass value="0.02"/>
+    <inertia ixx="0.00005" iyy="0.00005" izz="0.00001" ixy="0" ixz="0" iyz="0"/>
   </inertial>
   <visual>
@@ -187,6 +187,5 @@
   <inertial>
     <origin xyz="-0.005346701893651634 0.008500459968431101 -8.326672684688674e-17" rpy="0 0 0"/>
-    <mass value="0.008194856226231374"/>
-    <inertia ixx="0.0" iyy="1e-06" izz="1e-06" ixy="0.0" iyz="0.0" ixz="-0.0"/>
+    <mass value="0.04"/> <inertia ixx="0.00001" iyy="0.00001" izz="0.00001" ixy="0" iyz="0" ixz="0"/>
   </inertial>
   <visual>
@@ -207,6 +206,5 @@
   <inertial>
     <origin xyz="-0.005346701893651551 -0.008499919116163546 0.0" rpy="0 0 0"/>
-    <mass value="0.008194856226231374"/>
-    <inertia ixx="0.0" iyy="1e-06" izz="1e-06" ixy="0.0" iyz="0.0" ixz="0.0"/>
+    <mass value="0.04"/> <inertia ixx="0.00001" iyy="0.00001" izz="0.00001" ixy="0" iyz="0" ixz="0"/>
   </inertial>
   <visual>
@@ -227,6 +225,5 @@
   <inertial>
     <origin xyz="0.005346701893651509 0.00850045996843099 0.0" rpy="0 0 0"/>
-    <mass value="0.008194856226231374"/>
-    <inertia ixx="0.0" iyy="1e-06" izz="1e-06" ixy="-0.0" iyz="0.0" ixz="0.0"/>
+    <mass value="0.04"/> <inertia ixx="0.00001" iyy="0.00001" izz="0.00001" ixy="0" iyz="0" ixz="0"/>
   </inertial>
   <visual>
@@ -247,6 +244,5 @@
   <inertial>
     <origin xyz="0.005346701893651579 -0.008499919116163601 0.0" rpy="0 0 0"/>
-    <mass value="0.008194856226231374"/>
-    <inertia ixx="0.0" iyy="1e-06" izz="1e-06" ixy="-0.0" iyz="0.0" ixz="0.0"/>
+    <mass value="0.04"/> <inertia ixx="0.00001" iyy="0.00001" izz="0.00001" ixy="0" iyz="0" ixz="0"/>
   </inertial>
   <visual>
